Commit message: disparity gap detection

File: src/f1tenth_simulator/racecar.xacro (robot description, xacro)
@@ -2,5 +2,5 @@
 <!-- A simple model of the racecar for rviz -->
 <robot xmlns:xacro="http://www.ros.org/wiki/xacro" name="racecar">
-  <xacro:property name="wheelbase" value="0.3302" />
+  <xacro:property name="wheelbase" value="0.25" />
   <xacro:property name="width" value="0.2032" />
   <xacro:property name="height" value="0.1" />

Commit message: idk

File: src/f1tenth_simulator/racecar.xacro (robot description, xacro)
@@ -2,12 +2,12 @@
 <!-- A simple model of the racecar for rviz -->
 <robot xmlns:xacro="http://www.ros.org/wiki/xacro" name="racecar">
-  <xacro:property name="wheelbase" value="0.25" />
-  <xacro:property name="width" value="0.2032" />
-  <xacro:property name="height" value="0.1" />
+  <xacro:property name="wheelbase" value="0.3429" />
+  <xacro:property name="width" value="0.254" />
+  <xacro:property name="height" value="0.2159" />
   <xacro:property name="ground_offset" value="0.04" />
-  <xacro:property name="wheel_radius" value="0.0508" />
-  <xacro:property name="wheel_length" value="0.0381" />
+  <xacro:property name="wheel_radius" value="0.1" />
+  <xacro:property name="wheel_length" value="0.05" />
   <xacro:property name="laser_distance_from_base_link" value="0.275" />
-  <xacro:property name="laser_height" value="0.05" />
+  <xacro:property name="laser_height" value="0.1" />
   <xacro:property name="laser_radius" value="0.026" />
   <material name="black">
